Commit message: push changes

File: world/urdf/pr2.urdf (robot description, URDF)
Before this commit: robot pr2, 95 links, 94 joints
Links:
- link base_link: geometry collision mesh filename=package://pr2_description/meshes/base_v0/base_L.stl; visual mesh filename=package://pr2_description/meshes/base_v0/base.dae
- link bl_caster_l_wheel_link: geometry collision cylinder length=0.034 radius=0.074792; visual mesh filename=package://pr2_description/meshes/base_v0/wheel.dae
- link bl_caster_r_wheel_link: geometry collision cylinder length=0.034 radius=0.074792; visual mesh filename=package://pr2_description/meshes/base_v0/wheel.dae
- link bl_caster_rotation_link: geometry collision mesh filename=package://pr2_description/meshes/base_v0/caster_L.stl; visual mesh filename=package://pr2_description/meshes/base_v0/caster.stl
- link br_caster_l_wheel_link: geometry collision cylinder length=0.034 radius=0.074792; visual mesh filename=package://pr2_description/meshes/base_v0/wheel.dae
- link br_caster_r_wheel_link: geometry collision cylinder length=0.034 radius=0.074792; visual mesh filename=package://pr2_description/meshes/base_v0/wheel.dae
- link br_caster_rotation_link: geometry collision mesh filename=package://pr2_description/meshes/base_v0/caster_L.stl; visual mesh filename=package://pr2_description/meshes/base_v0/caster.stl
- link fl_caster_l_wheel_link: geometry collision cylinder length=0.034 radius=0.074792; visual mesh filename=package://pr2_description/meshes/base_v0/wheel.dae
- link fl_caster_r_wheel_link: geometry collision cylinder length=0.034 radius=0.074792; visual mesh filename=package://pr2_description/meshes/base_v0/wheel.dae
- link fl_caster_rotation_link: geometry collision mesh filename=package://pr2_description/meshes/base_v0/caster_L.stl; visual mesh filename=package://pr2_description/meshes/base_v0/caster.stl
- link fr_caster_l_wheel_link: geometry collision cylinder length=0.034 radius=0.074792; visual mesh filename=package://pr2_description/meshes/base_v0/wheel.dae
- link fr_caster_r_wheel_link: geometry collision cylinder length=0.034 radius=0.074792; visual mesh filename=package://pr2_description/meshes/base_v0/wheel.dae
- link fr_caster_rotation_link: geometry collision mesh filename=package://pr2_description/meshes/base_v0/caster_L.stl; visual mesh filename=package://pr2_description/meshes/base_v0/caster.stl
- link head_mount_link: geometry collision sphere radius=0.0005; visual mesh filename=package://pr2_description/meshes/sensors/kinect_prosilica_v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 scale=0.001 0.001 0.001
- link head_pan_link: geometry collision mesh filename=package://pr2_description/meshes/head_v0/head_pan_L.stl; visual mesh filename=package://pr2_description/meshes/head_v0/head_pan.dae
- link head_tilt_link: geometry collision mesh filename=package://pr2_description/meshes/head_v0/head_tilt_L.stl; visual mesh filename=package://pr2_description/meshes/head_v0/head_tilt.dae
- link l_elbow_flex_link: geometry collision mesh filename=package://pr2_description/meshes/upper_arm_v0/elbow_flex.stl; visual mesh filename=package://pr2_description/meshes/upper_arm_v0/elbow_flex.dae
- link l_forearm_link: geometry collision mesh filename=package://pr2_description/meshes/forearm_v0/forearm.stl; visual mesh filename=package://pr2_description/meshes/forearm_v0/forearm.dae
- link l_forearm_roll_link: geometry collision mesh filename=package://pr2_description/meshes/upper_arm_v0/forearm_roll_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; visual mesh filename=package://pr2_description/meshes/upper_arm_v0/forearm_roll.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
- link l_gripper_l_finger_link: geometry collision mesh filename=package://pr2_description/meshes/gripper_v0/l_finger.stl; visual mesh filename=package://pr2_description/meshes/gripper_v0/l_finger.dae
- link l_gripper_l_finger_tip_link: geometry collision mesh filename=package://pr2_description/meshes/gripper_v0/l_finger_tip.stl; visual mesh filename=package://pr2_description/meshes/gripper_v0/l_finger_tip.dae
- link l_gripper_palm_link: geometry collision mesh filename=package://pr2_description/meshes/gripper_v0/gripper_palm.stl; visual mesh filename=package://pr2_description/meshes/gripper_v0/gripper_palm.dae
- link l_gripper_r_finger_link: geometry collision mesh filename=package://pr2_description/meshes/gripper_v0/l_finger.stl; visual mesh filename=package://pr2_description/meshes/gripper_v0/l_finger.dae
- link l_gripper_r_finger_tip_link: geometry collision mesh filename=package://pr2_description/meshes/gripper_v0/l_finger_tip.stl; visual mesh filename=package://pr2_description/meshes/gripper_v0/l_finger_tip.dae
- link l_shoulder_lift_link: geometry collision mesh filename=package://pr2_description/meshes/shoulder_v0/shoulder_lift.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; visual mesh filename=package://pr2_description/meshes/shoulder_v0/shoulder_lift.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
- link l_shoulder_pan_link: geometry collision mesh filename=package://pr2_description/meshes/shoulder_v0/shoulder_pan.s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; visual mesh filename=package://pr2_description/meshes/shoulder_v0/shoulder_pan.d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
- link l_upper_arm_link: geometry collision mesh filename=package://pr2_description/meshes/upper_arm_v0/upper_arm.stl; visual mesh filename=package://pr2_description/meshes/upper_arm_v0/upper_arm.dae
- link l_upper_arm_roll_link: geometry collision mesh filename=package://pr2_description/meshes/shoulder_v0/upper_arm_roll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; visual mesh filename=package://pr2_description/meshes/shoulder_v0/upper_arm_roll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
- link l_wrist_flex_link: geometry collision mesh filename=package://pr2_description/meshes/forearm_v0/wrist_flex.stl; visual mesh filename=package://pr2_description/meshes/forearm_v0/wrist_flex.dae
- link l_wrist_roll_link: geometry collision mesh filename=package://pr2_description/meshes/forearm_v0/wrist_roll_L.stl; visual mesh filename=package://pr2_description/meshes/forearm_v0/wrist_roll.stl
- link laser_tilt_mount_link: geometry collision mesh filename=package://pr2_description/meshes/tilting_laser_v0/tilting_h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; visual mesh filename=package://pr2_description/meshes/tilting_laser_v0/tilting_h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
- link r_elbow_flex_link: geometry collision mesh filename=package://pr2_description/meshes/upper_arm_v0/elbow_flex.stl; visual mesh filename=package://pr2_description/meshes/upper_arm_v0/elbow_flex.dae
- link r_forearm_link: geometry collision mesh filename=package://pr2_description/meshes/forearm_v0/forearm.stl; visual mesh filename=package://pr2_description/meshes/forearm_v0/forearm.dae
- link r_forearm_roll_link: geometry collision mesh filename=package://pr2_description/meshes/upper_arm_v0/forearm_roll_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; visual mesh filename=package://pr2_description/meshes/upper_arm_v0/forearm_roll.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
- link r_gripper_l_finger_link: geometry collision mesh filename=package://pr2_description/meshes/gripper_v0/l_finger.stl; visual mesh filename=package://pr2_description/meshes/gripper_v0/l_finger.dae
- link r_gripper_l_finger_tip_link: geometry collision mesh filename=package://pr2_description/meshes/gripper_v0/l_finger_tip.stl; visual mesh filename=package://pr2_description/meshes/gripper_v0/l_finger_tip.dae
- link r_gripper_palm_link: geometry collision mesh filename=package://pr2_description/meshes/gripper_v0/gripper_palm.stl; visual mesh filename=package://pr2_description/meshes/gripper_v0/gripper_palm.dae
- link r_gripper_r_finger_link: geometry collision mesh filename=package://pr2_description/meshes/gripper_v0/l_finger.stl; visual mesh filename=package://pr2_description/meshes/gripper_v0/l_finger.dae
- link r_gripper_r_finger_tip_link: geometry collision mesh filename=package://pr2_description/meshes/gripper_v0/l_finger_tip.stl; visual mesh filename=package://pr2_description/meshes/gripper_v0/l_finger_tip.dae
- link r_shoulder_lift_link: geometry collision mesh filename=package://pr2_description/meshes/shoulder_v0/shoulder_lift.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; visual mesh filename=package://pr2_description/meshes/shoulder_v0/shoulder_lift.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
- link r_shoulder_pan_link: geometry collision mesh filename=package://pr2_description/meshes/shoulder_v0/shoulder_pan.s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; visual mesh filename=package://pr2_description/meshes/shoulder_v0/shoulder_pan.d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
- link r_upper_arm_link: geometry collision mesh filename=package://pr2_description/meshes/upper_arm_v0/upper_arm.stl; visual mesh filename=package://pr2_description/meshes/upper_arm_v0/upper_arm.dae
- link r_upper_arm_roll_link: geometry collision mesh filename=package://pr2_description/meshes/shoulder_v0/upper_arm_roll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; visual mesh filename=package://pr2_description/meshes/shoulder_v0/upper_arm_roll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
- link r_wrist_flex_link: geometry collision mesh filename=package://pr2_description/meshes/forearm_v0/wrist_flex.stl; visual mesh filename=package://pr2_description/meshes/forearm_v0/wrist_flex.dae
- link r_wrist_roll_link: geometry collision mesh filename=package://pr2_description/meshes/forearm_v0/wrist_roll_L.stl; visual mesh filename=package://pr2_description/meshes/forearm_v0/wrist_roll.stl
- link torso_lift_link: geometry collision mesh filename=package://pr2_description/meshes/torso_v0/torso_lift_L.stl; visual mesh filename=package://pr2_description/meshes/torso_v0/torso_lift.dae
